File: docs/schematic/ets-breakout.kicad_sch (KiCad schematic)
At the start: 26 parts, among them J5 QSE-040-01-L-D-A, K0 MCX-J-P-H-ST-TH1, K1 MCX-J-P-H-ST-TH1, K10 MCX-J-P-H-ST-TH1, K11 MCX-J-P-H-ST-TH1, K12 MCX-J-P-H-ST-TH1, K13 MCX-J-P-H-ST-TH1, K14 MCX-J-P-H-ST-TH1, K15 MCX-J-P-H-ST-TH1, K16 MCX-J-P-H-ST-TH1, K17 MCX-J-P-H-ST-TH1, K18 MCX-J-P-H-ST-TH1, K19 MCX-J-P-H-ST-TH1, K2 MCX-J-P-H-ST-TH1, K20 MCX-J-P-H-ST-TH1, K21 MCX-J-P-H-ST-TH1, K22 MCX-J-P-H-ST-TH1, K23 MCX-J-P-H-ST-TH1, K3 MCX-J-P-H-ST-TH1, K4 MCX-J-P-H-ST-TH1, K5 MCX-J-P-H-ST-TH1, K6 MCX-J-P-H-ST-TH1, K7 MCX-J-P-H-ST-TH1, K8 MCX-J-P-H-ST-TH1, K9 MCX-J-P-H-ST-TH1

Commit message: update after engineering review
Parts:
- removed IV, K0, K1, K10, K11, K12, K13, K14, K15, K16, K17, K18, K19, K2, K20, K21, K22, K23, K3, K4, K5, K6, K7, K8, K9: MCX-J-P-H-ST-TH1, symbol ets:COAX_JACK
- added J10, J11, J12, J13, J14, J15, J16, J17, J18, J19, J20, J21, J22, J23, J24, J25, J26, J27, J28, J29, J30, J6, J7, J8, J9: MCX-J-P-H-ST-TH1, symbol ets:COAX_JACK
Connections:
- net GNDA: now also J10.2 (SHLD), J11.2 (SHLD), J12.2 (SHLD), J13.2 (SHLD), J14.2 (SHLD), J15.2 (SHLD), J16.2 (SHLD), J17.2 (SHLD), J18.2 (SHLD), J19.2 (SHLD), J20.2 (SHLD), J21.2 (SHLD), J22.2 (SHLD), J23.2 (SHLD), J24.2 (SHLD), J25.2 (SHLD), J26.2 (SHLD), J27.2 (SHLD), J28.2 (SHLD), J29.2 (SHLD), J30.2 (SHLD), J6.2 (SHLD), J7.2 (SHLD), J8.2 (SHLD), J9.2 (SHLD)
- net IV: now also J30.1 (SIG)
- net SIPM_K0: now also J6.1 (SIG)
- net SIPM_K1: now also J7.1 (SIG)
- net SIPM_K10: now also J16.1 (SIG)
- net SIPM_K11: now also J17.1 (SIG)
- net SIPM_K12: now also J18.1 (SIG)
- net SIPM_K13: now also J19.1 (SIG)
- net SIPM_K14: now also J20.1 (SIG)
- net SIPM_K15: now also J21.1 (SIG)
- net SIPM_K16: now also J22.1 (SIG)
- net SIPM_K17: now also J23.1 (SIG)
- net SIPM_K18: now also J24.1 (SIG)
- net SIPM_K19: now also J25.1 (SIG)
- net SIPM_K2: now also J8.1 (SIG)
- net SIPM_K20: now also J26.1 (SIG)
- net SIPM_K21: now also J27.1 (SIG)
- net SIPM_K22: now also J28.1 (SIG)
- net SIPM_K23: now also J29.1 (SIG)
- net SIPM_K3: now also J9.1 (SIG)
- net SIPM_K4: now also J10.1 (SIG)
- net SIPM_K5: now also J11.1 (SIG)
- net SIPM_K6: now also J12.1 (SIG)
- net SIPM_K7: now also J13.1 (SIG)
- net SIPM_K8: now also J14.1 (SIG)
- net SIPM_K9: now also J15.1 (SIG)
